File: Hardware/Basic/Top/MV500-BASIC-TOP.sch (EAGLE design)
At the start: 19 parts, among them U2 NRF52832_MODULE_MDBT42

Commit message: Added OLED and SD Card
Parts:
- added C13, C15, C17, C18, C19: 2.2uF, LinnesLab-Passives:CAPACITOR0402
- added C16: 10uF, LinnesLab-Passives:CAPACITOR0603
- added R6: 10k, LinnesLab-Passives:RESISTOR0603
- added R7: 390k, LinnesLab-Passives:RESISTOR0603
- added SD2: (no value), LinnesLab-Connectors:MICROSD
- added U3: (no value), LinnesLab-Displays:DISP_OLED_UG-2864HSWEG01-NO-WRAPAROUND
Connections:
- new net CD1: SD2.CARD_DETECT
- new net CD2: SD2.CARD_DETECT1
- new net CS.OLED: U3./CS
- new net DC.OLED: U3.DC/I2C_SA0
- new net N$1: R6.2, U3.BS1
- new net N$13: C16.2, U3.VCC
- new net N$15: C18.2, U3.VCOMH
- new net N$2: R7.1, U3.IREF
- new net N$3: C13.2, U3.C2P
- new net N$5: C13.1, U3.C2N
- new net N$7: C15.2, U3.C1P
- new net N$8: C15.1, U3.C1N
- new net RESET.OLED: U3./RES
- new net SD.CS: SD2.CS
- net 3.3V: now also C17.2, C19.2, SD2.VDD, U3.VBAT, U3.VDD
- net GND: now also C16.1, C17.1, C18.1, C19.1, R6.1, R7.2, SD2.GND, SD2.GND1, SD2.VSS, U3.BS0, U3.BS2, U3.NC(GND)@1, U3.NC(GND)@2, U3.VLSS, U3.VSS
- net MISO: now also SD2.DATA_OUT
- net MOSI: now also SD2.DATA_IN, U3.D1/SPI_SDIN/I2C_SDA
- net SCK: now also SD2.SCLK, U3.D0/SPI_SCLK/I2C_SCK
Other:
- note added: "Connect MISO, MOSI, and SCK to appropriate pins on microcontroller. Those are SPI pins and are generally prespecified. You have more flexibility with the SD.CS pin."
- note added: "OLED"
- moved on the sheet: C10, C11, C12, C7, C8, C9, L2, LED3, LED4, R3, R4, SW3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

Commit message: Updated TOP schematic
Parts:
- added C2, C5, C6: 1u, LinnesLab-Passives:CAPACITOR0603
- added C20, C21: 4.7u, LinnesLab-Passives:CAPACITOR0603
- added CHRG2: MCP73831, LinnesLab-Power:MCP73831
- added D4, D5: (no value), LinnesLab-DiscreteSemi:SCHOTTKY-USC
- added J2: (no value), LinnesLab-Connectors:CONN_02
- added LDO2: MIC5504, LinnesLab-Power:MIC5504
- added R11: (no value), LinnesLab-Passives:RESISTOR0603
- added R12, R13, R14, R15: 100k, LinnesLab-Passives:RESISTOR0603
- added R8, R9: 10k, LinnesLab-Passives:RESISTOR0603
- added SW1, SW2: SWITCH.MOM, LinnesLab-Switches:SWITCH.MOM
- added U4: PCF8523, LinnesLab-Clocks:PCF8523
- added USB2: USB.MICRO-BIGGERPADS, LinnesLab-Connectors:USB.MICRO-BIGGERPADS
- added XTAL3: 32.7680kHz, LinnesLab-Clocks:CRYSTALECS-.327-12.5-12-C-TR
Connections:
- new net BATT: R13.1, R14.2
- new net CHRG.STAT: CHRG2.STAT, R12.1
- new net N$16: SW1.3, SW1.4
- new net N$17: CHRG2.PROG, R11.2
- new net N$18: SW2.3, SW2.4
- new net N$19: U4.OSCO, XTAL3.1
- new net N$20: U4.OSCI, XTAL3.2
- new net SW1: SW1.1, SW2.1
- new net USB+: USB2.D+
- new net USB-: USB2.D-
- new net VBATT: U4.VBAT
- new net VIN: C21.2, C5.2, CHRG2.VIN, D4.C, D5.C, LDO2.EN, LDO2.IN, R12.2
- new net VLIPO: C20.1, CHRG2.VBAT, D4.A, J2.2, R13.2
- new net V_USB: D5.A, USB2.V+
- net 3.3V: now also C2.1, C6.1, LDO2.OUT, R15.2, R8.2, R9.2, U4.VDD
- net GND: now also C2.2, C20.2, C21.1, C5.1, C6.2, CHRG2.VSS, J2.1, LDO2.GND, R11.1, R14.1, R15.1, U4.VSS, USB2.GND, USB2.SHIELD
- net SCL: now also R8.1, U4.SCL
- net SDA: now also R9.1, U4.SDA
Other:
- note added: "Back-up battery if desired"
- note added: "Buttons"
- note added: "Cortex Debugger/ Programmer"
- note added: "Digital Outputs CS.OLED RESET.OLED DC.OLED Digital Inputs 3x buttons Charge Status Analog Inputs Battery Monitor Analog Outputs"
- note added: "I2C Address = 0x68h"
- note added: "Power Management"
- note added: "Real-Time Clock"
- note added: "SD Card"
- note added: "nRF52832 Module"
- moved on the sheet: C10, C11, C12, C13, C14, C15, C16, C17, C18, C19, C7, C8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

Commit message: Top Schematic
Parts:
- added C22: 100n, LinnesLab-Passives:CAPACITOR0603
- added C23, C24: 47p, LinnesLab-Passives:CAPACITOR0603
- added JP2: (no value), LinnesLab-Switches:JUMPER-SMT_2_NO_SILK
- added LED5: RED, LinnesLab-LED:LED0603
- added LED6: YELLOW, LinnesLab-LED:LED0603
- added R1, R2: 0, LinnesLab-Passives:RESISTOR0603
- added R17, R18: 27, LinnesLab-Passives:RESISTOR0603
- added R19, R20: 1k, LinnesLab-Passives:RESISTOR0603
- added U5: FT231XS, LinnesLab-DigitalIC:FT231XS
- R8, R9: value 10k -> 10K
Connections:
- removed net RXD: U2.P0.08
- removed net TXD: U2.P0.06
- removed net VBATT: U4.VBAT
- new net !CTS: JP2.2, U5.!CTS
- new net FT3V3: U5.3V3OUT
- new net N$25: R17.2, U5.USBDM
- new net N$26: R18.2, U5.USBDP
- new net N$27: LED5.C, R19.2
- new net N$28: LED6.C, R20.2
- new net RXD_FT: R2.1, U5.RXD
- new net RXD_NRF: R1.2, U2.P0.08
- new net RXLED: R19.1, U5.CBUS1
- new net TXD_FT: R1.1, U5.TXD
- new net TXD_NRF: R2.2, U2.P0.06
- new net TXLED: R20.1, U5.CBUS2
- net 3.3V: now also C22.2, LED5.A, LED6.A, R8.1, R9.1, U5.!RESET, U5.VCCIO; no longer R8.2, R9.2
- net DTR: now also U5.!DTR
- net GND: now also C22.1, C23.2, C24.1, JP2.1, U5.GND@16, U5.GND@6
- net SCL: now also R9.2; no longer R8.1
- net SDA: now also R8.2; no longer R9.1
- net USB+: now also C23.1, R18.1
- net USB-: now also C24.2, R17.1
- net V_USB: now also U5.VCC
Other:
- note added: "FTDI Serial-to-USB Converter"
- note added: "I don't remember if CTS needs to be grounded or left floating so here's a jumper to ground so it can be configued either way dynamically."
- note added: "NOTES Digital Outputs CS.OLED RESET.OLED DC.OLED Digital Inputs 3x buttons Charge Status Analog Inputs Battery Monitor Analog Outputs"
- note added: "TXD goes to RX on the other device RXD goes to TX on the other device"
- note removed: "Digital Outputs CS.OLED RESET.OLED DC.OLED Digital Inputs 3x buttons Charge Status Analog Inputs Battery Monitor Analog Outputs"
- moved on the sheet: C10, C11, C12, C13, C14, C15, C16, C17, C18, C19, C7, C8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

Commit message: Updated Top Schematic
Connections:
- removed net BATT: R13.1, R14.2
- removed net CD1: SD2.CARD_DETECT
- removed net CHRG.STAT: CHRG2.STAT, R12.1
- removed net CS.OLED: U3./CS
- removed net DC.OLED: U3.DC/I2C_SA0
- removed net RESET.OLED: U3./RES
- removed net SD.CS: SD2.CS
- removed net SW1: SW1.1, SW2.1
- new net A4/BATT: R13.1, R14.2, U2.P0.28/AIN4
- new net A6/TIA: U2.P0.30/AIN6
- new net A7/PPG: U2.P0.31/AIN7
- new net D11/SW1: SW1.1, U2.P0.11
- new net D15/SW2: SW2.1, U2.P0.15
- new net D16/CS.OLED: U2.P0.16, U3./CS
- new net D27/CHRG.STATUS: CHRG2.STAT, R12.1, U2.P0.27
- new net D29/LED.CTRL: U2.P0.29/AIN5
- new net D3/RESET.OLED: U2.P0.03/AIN1, U3./RES
- new net D4/DC.OLED: U2.P0.04/AIN2, U3.DC/I2C_SA0
- new net D5/CD1: SD2.CARD_DETECT, U2.P0.05/AIN3
- new net D7/SD.CS: SD2.CS, U2.P0.07
Other:
- note added: "Digital Output"
- moved on the sheet: C10, C11, C12, C7, C8, C9, L2, LED3, LED4, R3, R4, R8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
